Commit message: ver_0726_控制器力矩上不去

File: src/robot_model/urdf/robot.xacro (robot description, xacro)
@@ -3,15 +3,15 @@
     xmlns:xacro="http://ros.org/wiki/xacro">
     <!-- 计算惯性矩阵xacro -->
-    <xacro:include filename="inertial.xacro"/>
+    <!-- <xacro:include filename="inertial.xacro"/> -->
     <xacro:property name="pi" value="3.1415926"/>
-    <xacro:property name="base_link_mass" value="0.2"/>
+    <xacro:property name="base_link_mass" value="0.1"/>
     <xacro:property name="base_link_length" value="0.3"/>
     <xacro:property name="base_link_width" value="0.15"/>
     <xacro:property name="base_link_height" value="0.025"/>
-    <xacro:property name="wheel_active_mass" value="0.1"/>
+    <xacro:property name="wheel_active_mass" value="0.05"/>
     <xacro:property name="wheel_active_radius" value="0.12"/>
     <xacro:property name="wheel_active_width" value="0.05"/>
     <xacro:property name="wheel_position_biasY" value="${base_link_width/2 + wheel_active_width/2 + 0.005}"/>
-    <xacro:property name="wheel_passive_mass" value="0.1"/>
+    <xacro:property name="wheel_passive_mass" value="0.05"/>
     <xacro:property name="wheel_passive_radius" value="${(wheel_active_radius - base_link_height/2)/2}"/>
     <xacro:property name="wheel_passive_position_biasZ" value="${wheel_active_radius/2+base_link_height/2}"/>
@@ -158,9 +158,9 @@
             <child link="wheel_passive_${position}"/>
             <origin xyz="${-base_link_length/2} ${posflag * wheel_position_biasY} ${-wheel_passive_position_biasZ}"/>
-            <axis xyz="1 1 0"/>
+            <axis xyz="0 1 0"/>
         </joint>
         <gazebo reference="wheel_passive_${position}">
-            <mu1 value="200"/>
-            <mu2 value="100"/>
+            <mu1 value="0.5"/>
+            <mu2 value="0.1"/>
             <material>Gazebo/Yellow</material>
         </gazebo>
@@ -178,4 +178,29 @@
     <xacro:wheel_passive posflag="1" position="left"/>
     <xacro:wheel_passive posflag="-1" position="right"/>
+    <link name="imu_link">
+        <visual>
+            <geometry>
+                <box size="${base_link_length/2} ${base_link_width/2} ${base_link_height/2}" />
+            </geometry>
+            <origin xyz="0 0 0" rpy="0 0 0" />
+            <material name="green"/>
+        </visual>
+        <collision>
+            <geometry>
+                <box size="${base_link_length/2} ${base_link_width/2} ${base_link_height/2}" />
+            </geometry>
+            <origin xyz="0 0 0" rpy="0 0 0" />
+            <material name="green"/>
+        </collision>
+        <xacro:Box_inertial_matrix m="${base_link_mass/4}" l="${base_link_length/2}" w="${base_link_width/2}" h="${base_link_height/2}"/>
+    </link>
+    <gazebo reference="imu_link">
+        <material>Gazebo/Green</material>
+    </gazebo>
+    <joint name="imu2base" type="fixed">
+        <parent link="base_link"/>
+        <child link="imu_link"/>
+        <origin xyz="0 0 ${base_link_width/4 + base_link_height/2}" rpy="${pi/2} 0 0" />
+    </joint>
     <gazebo>
         <plugin name="gazebo_ros_control" filename="libgazebo_ros_control.so">

Commit message: ver_0726_控制完成

File: src/robot_model/urdf/robot.xacro (robot description, xacro)
@@ -5,13 +5,13 @@
     <!-- <xacro:include filename="inertial.xacro"/> -->
     <xacro:property name="pi" value="3.1415926"/>
-    <xacro:property name="base_link_mass" value="0.1"/>
+    <xacro:property name="base_link_mass" value="0.2"/>
     <xacro:property name="base_link_length" value="0.3"/>
     <xacro:property name="base_link_width" value="0.15"/>
     <xacro:property name="base_link_height" value="0.025"/>
-    <xacro:property name="wheel_active_mass" value="0.05"/>
+    <xacro:property name="wheel_active_mass" value="0.1"/>
     <xacro:property name="wheel_active_radius" value="0.12"/>
     <xacro:property name="wheel_active_width" value="0.05"/>
     <xacro:property name="wheel_position_biasY" value="${base_link_width/2 + wheel_active_width/2 + 0.005}"/>
-    <xacro:property name="wheel_passive_mass" value="0.05"/>
+    <xacro:property name="wheel_passive_mass" value="0.1"/>
     <xacro:property name="wheel_passive_radius" value="${(wheel_active_radius - base_link_height/2)/2}"/>
     <xacro:property name="wheel_passive_position_biasZ" value="${wheel_active_radius/2+base_link_height/2}"/>
@@ -114,10 +114,10 @@
             <parent link="base_link"/>
             <child link="wheel_active_${position}"/>
-            <origin xyz="${base_link_length/2} ${posflag * wheel_position_biasY} 0"/>
+            <origin xyz="${-base_link_length/2} ${posflag * wheel_position_biasY} 0"/>
             <axis xyz="0 1 0"/>
         </joint>
         <gazebo reference="wheel_active_${position}">
             <mu1 value="200"/>
-            <mu2 value="100"/>
+            <mu2 value="200"/>
             <material>Gazebo/Red</material>
         </gazebo>
@@ -157,10 +157,10 @@
             <parent link="base_link"/>
             <child link="wheel_passive_${position}"/>
-            <origin xyz="${-base_link_length/2} ${posflag * wheel_position_biasY} ${-wheel_passive_position_biasZ}"/>
+            <origin xyz="${base_link_length/2} ${posflag * wheel_position_biasY} ${-wheel_passive_position_biasZ}"/>
             <axis xyz="0 1 0"/>
         </joint>
         <gazebo reference="wheel_passive_${position}">
-            <mu1 value="0.5"/>
-            <mu2 value="0.1"/>
+            <mu1 value="0.05"/>
+            <mu2 value="0.025"/>
             <material>Gazebo/Yellow</material>
         </gazebo>
