Commit message: ver_0730_车体模型修改

File: src/robot_model/urdf/imu.xacro (robot description, xacro)
@@ -10,5 +10,5 @@
             <plugin filename="libgazebo_ros_imu_sensor.so" name="imu_plugin">
                 <topicName>/imu/data</topicName>
-                <updateRateHZ>50.0</updateRateHZ>
+                <updateRateHZ>20.0</updateRateHZ>
                 <gaussianNoise>0</gaussianNoise>
                 <xyzOffset>0 0 0</xyzOffset>

File: src/robot_model/urdf/robot.xacro (robot description, xacro)
@@ -6,10 +6,10 @@
     <xacro:property name="pi" value="3.1415926"/>
     <xacro:property name="base_link_mass" value="0.2"/>
-    <xacro:property name="base_link_length" value="0.3"/>
-    <xacro:property name="base_link_width" value="0.15"/>
-    <xacro:property name="base_link_height" value="0.025"/>
+    <xacro:property name="base_link_length" value="1"/>
+    <xacro:property name="base_link_width" value="0.5"/>
+    <xacro:property name="base_link_height" value="0.05"/>
     <xacro:property name="wheel_active_mass" value="0.1"/>
-    <xacro:property name="wheel_active_radius" value="0.12"/>
-    <xacro:property name="wheel_active_width" value="0.05"/>
+    <xacro:property name="wheel_active_radius" value="0.5"/>
+    <xacro:property name="wheel_active_width" value="0.1"/>
     <xacro:property name="wheel_position_biasY" value="${base_link_width/2 + wheel_active_width/2 + 0.005}"/>
     <xacro:property name="wheel_passive_mass" value="0.1"/>
